File: C64 Stereo SID.kicad_pcb (KiCad board)
At the start: 2 copper layers, 48.9 x 41.9 mm, 22 parts, among them J1 EXT_IN_SEL1, J2 EXT_IN_SEL2, J3 AUD_OUT, J4 ~CS, Q1 2N2222, U1 MOS_6581, U2 MOS_6581

Commit message: Updated gerbers and added images
Other:
- outline, holes or cut-outs redrawn
- board text added: "Revision B"
Changed lines of the file:
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@@
     (area 88.9 93.64 154.305001 151.130001)
     (thickness 1.6)
-    (drawings 60)
+    (drawings 61)
     (tracks 276)
     (zones 0)
@@
     )
   )
+  (gr_line (start 147.955 99.06) (end 147.955 138.43) (angle 90) (layer Edge.Cuts) (width 0.15))
+  (gr_line (start 100.33 97.79) (end 146.685 97.79) (angle 90) (layer Edge.Cuts) (width 0.15))
+  (gr_line (start 99.06 138.43) (end 99.06 99.06) (angle 90) (layer Edge.Cuts) (width 0.15))
+  (gr_line (start 146.685 139.7) (end 100.33 139.7) (angle 90) (layer Edge.Cuts) (width 0.15))
+  (gr_arc (start 146.685 99.06) (end 146.685 97.79) (angle 90) (layer Edge.Cuts) (width 0.15))
+  (gr_arc (start 100.33 99.06) (end 99.06 99.06) (angle 90) (layer Edge.Cuts) (width 0.15))
+  (gr_arc (start 146.685 138.43) (end 147.955 138.43) (angle 90) (layer Edge.Cuts) (width 0.15))
+  (gr_arc (start 100.33 138.43) (end 100.33 139.7) (angle 90) (layer Edge.Cuts) (width 0.15))
+  (gr_text "Revision B" (at 103.505 137.16) (layer B.SilkS)
+    (effects (font (size 0.7 0.7) (thickness 0.1)) (justify mirror))
+  )
   (gr_text github.com/tebl (at 135.89 137.16) (layer B.SilkS)
     (effects (font (size 0.8 0.8) (thickness 0.15)) (justify mirror))
@@
     (effects (font (size 1 1) (thickness 0.15)))
   )
-  (gr_line (start 147.32 97.79) (end 147.955 97.79) (angle 90) (layer Edge.Cuts) (width 0.15))
-  (gr_line (start 147.955 139.7) (end 147.32 139.7) (angle 90) (layer Edge.Cuts) (width 0.15))
-  (gr_line (start 147.955 139.065) (end 147.955 139.7) (angle 90) (layer Edge.Cuts) (width 0.15))
-  (gr_line (start 99.06 139.065) (end 99.06 139.7) (angle 90) (layer Edge.Cuts) (width 0.15))
-  (gr_line (start 147.955 139.065) (end 147.955 97.79) (angle 90) (layer Edge.Cuts) (width 0.15))
-  (gr_line (start 99.06 139.7) (end 147.32 139.7) (angle 90) (layer Edge.Cuts) (width 0.15))
-  (gr_line (start 99.06 97.79) (end 99.06 139.065) (angle 90) (layer Edge.Cuts) (width 0.15))
-  (gr_line (start 147.32 97.79) (end 99.06 97.79) (angle 90) (layer Edge.Cuts) (width 0.15))
   (segment (start 121.92 136.525) (end 121.92 138.43) (width 0.25) (layer F.Cu) (net 0))
   (via (at 121.92 136.525) (size 0.6) (drill 0.4) (layers F.Cu B.Cu) (net 0))

Commit message: Fixed missing trace on the revision B boards
Parts:
- J1, J2: footprint Pin_Headers:Pin_Header_Straight_1x03_Pitch2.54mm -> Pin_Headers:Pin_Header_Straight_1x02_Pitch2.54mm
Routing:
- net Net-(D1-Pad1): track 20.5 -> 43.9 mm
Other:
- board text added: "EXT_IN_SEL1/2 1-2"
- board text added: "Link R2, leave R3 empty for Stereo SID."
- board text removed: "EXT_IN_SEL1/2 1-2 2-3"

Commit message: Revised pin headers brought out
Parts:
- removed J2: EXT_IN_SEL2, Pin_Headers:Pin_Header_Straight_1x02_Pitch2.54mm
- J3: footprint Pin_Headers:Pin_Header_Straight_1x03_Pitch2.54mm -> Pin_Headers:Pin_Header_Straight_1x02_Pitch2.54mm
Connections:
- J3 pad 1: AUD_L -> AUD_R
- U2 pad 26: EXT_IN2 -> (no net)
Routing:
- net AUD_L: track 70.7 -> 14.7 mm, vias 4 -> 3
- net EXT_IN2: track 18.6 -> 0.00 mm
- net /EXT_IN: track 22.3 -> 12.9 mm
- net AUD_R: track 93.3 -> 91.3 mm
Other:
- board text added: "AUD_OUT 1- 2-"
- board text added: "Revision C"
- board text removed: "AUD_OUT 1- 2- 3-"
- board text removed: "EXT_IN"
- board text removed: "EXT_IN_SEL1/2 1-2"
- board text removed: "Left"
- board text removed: "Revision B"
