File: C64 Stereo SID.sch (KiCad schematic (older format))
At the start: 22 parts, among them J1 EXT_IN_SEL1, J2 EXT_IN_SEL2, J3 AUD_OUT, J4 ~CS, Q1 2N2222, U1 MOS_6581, U2 MOS_6581

Commit message: Fixed missing trace on the revision B boards
Parts:
- J1, J2: footprint Pin_Headers:Pin_Header_Straight_1x03_Pitch2.54mm -> Pin_Headers:Pin_Header_Straight_1x02_Pitch2.54mm; symbol Conn_01x03 -> Conn_01x02
Connections:
- net GND: no longer J1.3 (Pin_3), J2.3 (Pin_3)
Other:
- note added: "1-2 Stereo SID\n2-3 Pseudo stareo"
- note added: "B"
- note added: "C64 Stereo SID"
- note added: "There are many Stereo SID boards, but this one is mine and it's out there for all who'd\nwant one, those that don't haven't heard axelf SID file played in glorious stereo on a real\nCommodore 64."
- note added: "This section downmixes both SID outputs\ninto a single signal output on the regular\naudio output (5 or 8 pin DIN). Leave out\nR3 and install a wire in R2 to make board\noperate in stereo mode."
- moved on the sheet: J4, R2, R3
Changed lines of the file:
@@
 EXT_IN
 $Comp
-L Conn_01x03 J1
+L Conn_01x02 J1
 U 1 1 5D1944E7
-P 6025 6825
-F 0 "J1" H 6025 7025 50  0000 C CNN
-F 1 "EXT_IN_SEL1" V 6125 6825 50  0000 C CNN
-F 2 "Pin_Headers:Pin_Header_Straight_1x03_Pitch2.54mm" H 6025 6825 50  0001 C CNN
-F 3 "" H 6025 6825 50  0001 C CNN
-	1    6025 6825
+P 6025 6725
+F 0 "J1" H 6025 6925 50  0000 C CNN
+F 1 "EXT_IN_SEL1" V 6125 6725 50  0000 C CNN
+F 2 "Pin_Headers:Pin_Header_Straight_1x02_Pitch2.54mm" H 6025 6725 50  0001 C CNN
+F 3 "" H 6025 6725 50  0001 C CNN
+	1    6025 6725
 	-1   0    0    -1
 $EndComp
@@
 EXT_IN
 $Comp
-L GND #PWR07
-U 1 1 5D19470F
-P 6300 7000
-F 0 "#PWR07" H 6300 6750 50  0001 C CNN
-F 1 "GND" H 6300 6850 50  0000 C CNN
-F 2 "" H 6300 7000 50  0001 C CNN
-F 3 "" H 6300 7000 50  0001 C CNN
-	1    6300 7000
-	-1   0    0    -1
-$EndComp
-$Comp
-L Conn_01x03 J2
+L Conn_01x02 J2
 U 1 1 5D194DC1
-P 6025 3050
-F 0 "J2" H 6025 3250 50  0000 C CNN
-F 1 "EXT_IN_SEL2" V 6125 3050 50  0000 C CNN
-F 2 "Pin_Headers:Pin_Header_Straight_1x03_Pitch2.54mm" H 6025 3050 50  0001 C CNN
-F 3 "" H 6025 3050 50  0001 C CNN
-	1    6025 3050
+P 6025 2950
+F 0 "J2" H 6025 3050 50  0000 C CNN
+F 1 "EXT_IN_SEL2" V 6125 2950 50  0000 C CNN
+F 2 "Pin_Headers:Pin_Header_Straight_1x02_Pitch2.54mm" H 6025 2950 50  0001 C CNN
+F 3 "" H 6025 2950 50  0001 C CNN
+	1    6025 2950
 	-1   0    0    -1
 $EndComp
@@
 Text Label 6675 2950 2    60   ~ 0
 EXT_IN
-$Comp
-L GND #PWR08
-U 1 1 5D194DCC
-P 6300 3225
-F 0 "#PWR08" H 6300 2975 50  0001 C CNN
-F 1 "GND" H 6300 3075 50  0000 C CNN
-F 2 "" H 6300 3225 50  0001 C CNN
-F 3 "" H 6300 3225 50  0001 C CNN
-	1    6300 3225
-	-1   0    0    -1
-$EndComp
 Text GLabel 6300 6825 2    60   Output ~ 0
 EXT_IN1
@@
 A4
 $Comp
-L GND #PWR09
+L GND #PWR07
 U 1 1 5D19627B
 P 4700 2600
-F 0 "#PWR09" H 4700 2350 50  0001 C CNN
+F 0 "#PWR07" H 4700 2350 50  0001 C CNN
 F 1 "GND" H 4700 2450 50  0000 C CNN
 F 2 "" H 4700 2600 50  0001 C CNN
@@
 	6700 2525 6800 2625
 $Comp
-L VDD #PWR010
+L VDD #PWR08
 U 1 1 5D1962A4
 P 6300 1150
-F 0 "#PWR010" H 6300 1000 50  0001 C CNN
+F 0 "#PWR08" H 6300 1000 50  0001 C CNN
 F 1 "VDD" H 6300 1300 50  0000 C CNN
 F 2 "" H 6300 1150 50  0001 C CNN
@@
 $EndComp
 $Comp
-L VCC #PWR011
+L VCC #PWR09
 U 1 1 5D1962AA
 P 6600 1525
-F 0 "#PWR011" H 6600 1375 50  0001 C CNN
+F 0 "#PWR09" H 6600 1375 50  0001 C CNN
 F 1 "VCC" H 6600 1675 50  0000 C CNN
 F 2 "" H 6600 1525 50  0001 C CNN
@@
 $EndComp
 $Comp
-L GND #PWR012
+L GND #PWR010
 U 1 1 5D1985DD
 P 9600 5525
-F 0 "#PWR012" H 9600 5275 50  0001 C CNN
+F 0 "#PWR010" H 9600 5275 50  0001 C CNN
 F 1 "GND" H 9600 5375 50  0000 C CNN
 F 2 "" H 9600 5525 50  0001 C CNN
@@
 	1    0    0    -1
 $EndComp
-Text GLabel 4850 3050 0    60   Output ~ 0
+Text GLabel 4850 2950 0    60   Output ~ 0
 ~CS2_IN
 $Comp
@@
 $EndComp
 $Comp
-L VDD #PWR013
+L VDD #PWR011
 U 1 1 5D19A465
 P 8850 1500
-F 0 "#PWR013" H 8850 1350 50  0001 C CNN
+F 0 "#PWR011" H 8850 1350 50  0001 C CNN
 F 1 "VDD" H 8850 1650 50  0000 C CNN
 F 2 "" H 8850 1500 50  0001 C CNN
@@
 $EndComp
 $Comp
-L GND #PWR014
+L GND #PWR012
 U 1 1 5D19BFF2
 P 8275 2650
-F 0 "#PWR014" H 8275 2400 50  0001 C CNN
+F 0 "#PWR012" H 8275 2400 50  0001 C CNN
 F 1 "GND" H 8275 2500 50  0000 C CNN
 F 2 "" H 8275 2650 50  0001 C CNN
@@
 $EndComp
 $Comp
-L GND #PWR015
+L GND #PWR013
 U 1 1 5D19C774
 P 7375 1775
-F 0 "#PWR015" H 7375 1525 50  0001 C CNN
+F 0 "#PWR013" H 7375 1525 50  0001 C CNN
 F 1 "GND" H 7375 1625 50  0000 C CNN
 F 2 "" H 7375 1775 50  0001 C CNN
@@
 $EndComp
 $Comp
-L GND #PWR016
+L GND #PWR014
 U 1 1 5D19CE76
 P 8000 2200
-F 0 "#PWR016" H 8000 1950 50  0001 C CNN
+F 0 "#PWR014" H 8000 1950 50  0001 C CNN
 F 1 "GND" H 8000 2050 50  0000 C CNN
 F 2 "" H 8000 2200 50  0001 C CNN
@@
 SID #1
 $Comp
-L VCC #PWR017
+L VCC #PWR015
 U 1 1 5D1ADB09
-P 4425 3075
-F 0 "#PWR017" H 4425 2925 50  0001 C CNN
-F 1 "VCC" H 4425 3225 50  0000 C CNN
-F 2 "" H 4425 3075 50  0001 C CNN
-F 3 "" H 4425 3075 50  0001 C CNN
-	1    4425 3075
+P 4425 2975
+F 0 "#PWR015" H 4425 2825 50  0001 C CNN
+F 1 "VCC" H 4425 3125 50  0000 C CNN
+F 2 "" H 4425 2975 50  0001 C CNN
+F 3 "" H 4425 2975 50  0001 C CNN
+	1    4425 2975
 	1    0    0    -1
 $EndComp
@@
 L Conn_01x02 J4
 U 1 1 5D1ADE1F
-P 5125 3050
-F 0 "J4" H 5125 3150 50  0000 C CNN
-F 1 "~CS" H 5125 2850 50  0000 C CNN
-F 2 "Pin_Headers:Pin_Header_Straight_1x02_Pitch2.54mm" H 5125 3050 50  0001 C CNN
-F 3 "" H 5125 3050 50  0001 C CNN
-	1    5125 3050
+P 5125 2950
+F 0 "J4" H 5125 3050 50  0000 C CNN
+F 1 "~CS" H 5125 2750 50  0000 C CNN
+F 2 "Pin_Headers:Pin_Header_Straight_1x02_Pitch2.54mm" H 5125 2950 50  0001 C CNN
+F 3 "" H 5125 2950 50  0001 C CNN
+	1    5125 2950
 	1    0    0    -1
 $EndComp
@@
 $EndComp
 $Comp
-L GND #PWR018
+L GND #PWR016
 U 1 1 5D430FD6
 P 8275 4050
-F 0 "#PWR018" H 8275 3800 50  0001 C CNN
+F 0 "#PWR016" H 8275 3800 50  0001 C CNN
 F 1 "GND" H 8275 3900 50  0000 C CNN
 F 2 "" H 8275 4050 50  0001 C CNN
@@
 $EndComp
 $Comp
-L GND #PWR019
+L GND #PWR017
 U 1 1 5D431AE6
 P 4100 1900
-F 0 "#PWR019" H 4100 1650 50  0001 C CNN
+F 0 "#PWR017" H 4100 1650 50  0001 C CNN
 F 1 "GND" H 4100 1750 50  0000 C CNN
 F 2 "" H 4100 1900 50  0001 C CNN
@@
 	6225 6725 6700 6725
 Wire Wire Line
-	6225 6925 6300 6925
-Wire Wire Line
-	6300 6925 6300 7000
-Wire Wire Line
 	6225 2950 6700 2950
 Wire Wire Line
-	6225 3150 6300 3150
-Wire Wire Line
-	6300 3150 6300 3225
-Wire Wire Line
 	6225 6825 6300 6825
 Wire Wire Line
@@
 	9600 5375 9600 5525
 Wire Wire Line
-	4850 3050 4925 3050
+	4850 2950 4925 2950
 Wire Wire Line
 	6225 1325 8275 1325
@@
 	675  3050 3700 3050
 Wire Wire Line
-	4425 3075 4425 3150
-Wire Wire Line
-	4425 3150 4925 3150
+	4425 2975 4425 3050
+Wire Wire Line
+	4425 3050 4925 3050
 Wire Wire Line
 	4650 1925 4775 1925
@@
 Text GLabel 6225 5100 2    60   Output ~ 0
 AUD_L
-Text GLabel 8025 5350 0    60   Input ~ 0
+Text GLabel 8025 5475 0    60   Input ~ 0
 AUD_R
-Text GLabel 8550 5250 2    60   Output ~ 0
+Text GLabel 8550 5375 2    60   Output ~ 0
 AUD_OUT
 Text GLabel 9350 2200 2    60   Output ~ 0
@@
 Wire Wire Line
 	10025 5275 10100 5275
-Text GLabel 8025 5150 0    60   Input ~ 0
+Text GLabel 8025 5275 0    60   Input ~ 0
 AUD_L
 $Comp
 L R R2
 U 1 1 5D4B59AE
-P 8250 5150
-F 0 "R2" V 8330 5150 50  0000 C CNN
-F 1 "1k" V 8250 5150 50  0000 C CNN
-F 2 "Resistors_THT:R_Axial_DIN0207_L6.3mm_D2.5mm_P10.16mm_Horizontal" V 8180 5150 50  0001 C CNN
-F 3 "" H 8250 5150 50  0001 C CNN
-	1    8250 5150
+P 8250 5275
+F 0 "R2" V 8330 5275 50  0000 C CNN
+F 1 "1k" V 8250 5275 50  0000 C CNN
+F 2 "Resistors_THT:R_Axial_DIN0207_L6.3mm_D2.5mm_P10.16mm_Horizontal" V 8180 5275 50  0001 C CNN
+F 3 "" H 8250 5275 50  0001 C CNN
+	1    8250 5275
 	0    1    1    0
 $EndComp
@@
 L R R3
 U 1 1 5D4B5DFF
-P 8250 5350
-F 0 "R3" V 8330 5350 50  0000 C CNN
-F 1 "1k" V 8250 5350 50  0000 C CNN
-F 2 "Resistors_THT:R_Axial_DIN0207_L6.3mm_D2.5mm_P10.16mm_Horizontal" V 8180 5350 50  0001 C CNN
-F 3 "" H 8250 5350 50  0001 C CNN
-	1    8250 5350
+P 8250 5475
+F 0 "R3" V 8330 5475 50  0000 C CNN
+F 1 "1k" V 8250 5475 50  0000 C CNN
+F 2 "Resistors_THT:R_Axial_DIN0207_L6.3mm_D2.5mm_P10.16mm_Horizontal" V 8180 5475 50  0001 C CNN
+F 3 "" H 8250 5475 50  0001 C CNN
+	1    8250 5475
 	0    1    1    0
 $EndComp
 Wire Wire Line
-	8475 5350 8400 5350
-Wire Wire Line
-	8475 5150 8475 5350
-Wire Wire Line
-	8475 5150 8400 5150
-Wire Wire Line
-	8550 5250 8475 5250
-Connection ~ 8475 5250
-Wire Wire Line
-	8100 5150 8025 5150
-Wire Wire Line
-	8025 5350 8100 5350
+	8475 5475 8400 5475
+Wire Wire Line
+	8475 5275 8475 5475
+Wire Wire Line
+	8475 5275 8400 5275
+Wire Wire Line
+	8550 5375 8475 5375
+Connection ~ 8475 5375
+Wire Wire Line
+	8100 5275 8025 5275
+Wire Wire Line
+	8025 5475 8100 5475
+Wire Notes Line
+	7500 5050 9025 5050
+Wire Notes Line
+	9025 5050 9025 5700
+Wire Notes Line
+	9025 5700 7500 5700
+Wire Notes Line
+	7500 5700 7500 5050
+Text Notes 7275 6225 0    60   ~ 0
+This section downmixes both SID outputs\ninto a single signal output on the regular\naudio output (5 or 8 pin DIN). Leave out\nR3 and install a wire in R2 to make board\noperate in stereo mode.
+Text Notes 7350 7500 0    60   ~ 0
+C64 Stereo SID
+Text Notes 10550 7650 0    60   ~ 0
+B
+Text Notes 6975 6850 0    60   ~ 0
+There are many Stereo SID boards, but this one is mine and it's out there for all who'd\nwant one, those that don't haven't heard axelf SID file played in glorious stereo on a real\nCommodore 64.
+Text Notes 8675 4250 0    60   ~ 0
+1-2 Stereo SID\n2-3 Pseudo stareo
 $EndSCHEMATC

Commit message: Revised pin headers brought out
Parts:
- removed J2: EXT_IN_SEL2, Pin_Headers:Pin_Header_Straight_1x02_Pitch2.54mm, symbol Conn_01x02
- J3: footprint Pin_Headers:Pin_Header_Straight_1x03_Pitch2.54mm -> Pin_Headers:Pin_Header_Straight_1x02_Pitch2.54mm; symbol Conn_01x03 -> Conn_01x02
Connections:
- net AUD_L: no longer J3.1 (Pin_1)
- net AUD_R: now also J3.1 (Pin_1); no longer J3.3 (Pin_3)
- net EXT_IN2: no longer names the net of U2.26 (EXT_IN)
- no-connect marks 2 -> 3
Other:
- note added: "C"
- note removed: "B"
Changed lines of the file:
@@
 Text Label 6675 6725 2    60   ~ 0
-EXT_IN
-$Comp
-L Conn_01x02 J2
-U 1 1 5D194DC1
-P 6025 2950
-F 0 "J2" H 6025 3050 50  0000 C CNN
-F 1 "EXT_IN_SEL2" V 6125 2950 50  0000 C CNN
-F 2 "Pin_Headers:Pin_Header_Straight_1x02_Pitch2.54mm" H 6025 2950 50  0001 C CNN
-F 3 "" H 6025 2950 50  0001 C CNN
-	1    6025 2950
-	-1   0    0    -1
-$EndComp
-Entry Wire Line
-	6800 2850 6700 2950
-Text Label 6675 2950 2    60   ~ 0
 EXT_IN
 Text GLabel 6300 6825 2    60   Output ~ 0
 EXT_IN1
-Text GLabel 6300 3050 2    60   Output ~ 0
-EXT_IN2
 $Comp
 L MOS_6581 U2
@@
 	0    1    1    0
 $EndComp
-Text GLabel 6225 1425 2    60   Input ~ 0
-EXT_IN2
 NoConn ~ 6225 1625
 NoConn ~ 6225 1725
@@
 L GND #PWR010
 U 1 1 5D1985DD
-P 9600 5525
-F 0 "#PWR010" H 9600 5275 50  0001 C CNN
-F 1 "GND" H 9600 5375 50  0000 C CNN
-F 2 "" H 9600 5525 50  0001 C CNN
-F 3 "" H 9600 5525 50  0001 C CNN
-	1    9600 5525
+P 9600 5625
+F 0 "#PWR010" H 9600 5375 50  0001 C CNN
+F 1 "GND" H 9600 5475 50  0000 C CNN
+F 2 "" H 9600 5625 50  0001 C CNN
+F 3 "" H 9600 5625 50  0001 C CNN
+	1    9600 5625
 	1    0    0    -1
 $EndComp
@@
 	6225 6725 6700 6725
 Wire Wire Line
-	6225 2950 6700 2950
-Wire Wire Line
 	6225 6825 6300 6825
-Wire Wire Line
-	6225 3050 6300 3050
 Wire Notes Line
 	6000 6825 6000 6725
@@
 	9200 2200 9350 2200
 Wire Wire Line
-	9600 5375 10100 5375
-Wire Wire Line
-	9600 5375 9600 5525
+	9600 5475 10100 5475
+Wire Wire Line
+	9600 5475 9600 5625
 Wire Wire Line
 	4850 2950 4925 2950
@@
 AUD_R
 $Comp
-L Conn_01x03 J3
+L Conn_01x02 J3
 U 1 1 5D44DABC
 P 10300 5375
 F 0 "J3" H 10300 5575 50  0000 C CNN
 F 1 "AUD_OUT" V 10400 5375 50  0000 C CNN
-F 2 "Pin_Headers:Pin_Header_Straight_1x03_Pitch2.54mm" H 10300 5375 50  0001 C CNN
+F 2 "Pin_Headers:Pin_Header_Straight_1x02_Pitch2.54mm" H 10300 5375 50  0001 C CNN
 F 3 "" H 10300 5375 50  0001 C CNN
 	1    10300 5375
 	1    0    0    -1
 $EndComp
-Text GLabel 10025 5275 0    60   Input ~ 0
-AUD_L
-Text GLabel 10025 5475 0    60   Input ~ 0
+Text GLabel 10025 5375 0    60   Input ~ 0
 AUD_R
 Wire Wire Line
-	10025 5475 10100 5475
-Wire Wire Line
-	10025 5275 10100 5275
+	10025 5375 10100 5375
 Text GLabel 8025 5275 0    60   Input ~ 0
 AUD_L
@@
 C64 Stereo SID
 Text Notes 10550 7650 0    60   ~ 0
-B
+C
 Text Notes 6975 6850 0    60   ~ 0
 There are many Stereo SID boards, but this one is mine and it's out there for all who'd\nwant one, those that don't haven't heard axelf SID file played in glorious stereo on a real\nCommodore 64.
 Text Notes 8675 4250 0    60   ~ 0
 1-2 Stereo SID\n2-3 Pseudo stareo
+NoConn ~ 6225 1425
 $EndSCHEMATC
